Commit message: feat: Integrate Robotiq-2f

File: ros2_ws/src/use_case_sim/urdf/task_env.urdf.xacro (robot description, xacro)
@@ -56,3 +56,22 @@
   <gazebo reference="table_link"><material>Gazebo/Wood</material></gazebo>
   <gazebo reference="plate_link"><material>Gazebo/DarkGrey</material></gazebo>
+  <xacro:include filename="$(find robotiq_description)/urdf/robotiq_2f_85_macro.urdf.xacro"/>
+  <xacro:robotiq_gripper name="RobotiqGripper" prefix="" parent="tool0" include_ros2_control="false">
+    <origin xyz="0 0 0" rpy="0 0 0"/>
+  </xacro:robotiq_gripper>
+  <ros2_control name="RobotiqGripperHardware" type="system">
+    <hardware>
+      <plugin>gazebo_ros2_control/GazeboSystem</plugin>
+    </hardware>
+    <joint name="robotiq_85_left_knuckle_joint">
+      <command_interface name="position">
+        <param name="min">0.0</param>
+        <param name="max">0.8</param>
+      </command_interface>
+      <state_interface name="position">
+        <param name="initial_value">0.0</param>
+      </state_interface>
+      <state_interface name="velocity"/>
+    </joint>
+  </ros2_control>
 </robot>

Commit message: feat: Add gripper and peg urdfs

File: ros2_ws/src/use_case_sim/urdf/task_env.urdf.xacro (robot description, xacro)
@@ -4,5 +4,5 @@
   <xacro:arg name="ur_type" default="ur10"/>
   <xacro:arg name="sim_gazebo" default="true"/>
-  <xacro:arg name="simulation_controllers" default="$(find ur_simulation_gazebo)/config/ur_controllers.yaml"/>
+  <xacro:arg name="simulation_controllers" default="$(find use_case_sim)/config/task_controllers.yaml"/>
   <xacro:include filename="$(find ur_description)/urdf/ur.urdf.xacro"/>
   <joint name="world_to_table" type="fixed">
@@ -65,11 +65,41 @@
     </hardware>
     <joint name="robotiq_85_left_knuckle_joint">
-      <command_interface name="position">
-        <param name="min">0.0</param>
-        <param name="max">0.8</param>
-      </command_interface>
-      <state_interface name="position">
-        <param name="initial_value">0.0</param>
-      </state_interface>
+      <command_interface name="position"/>
+      <state_interface name="position"><param name="initial_value">0.0</param></state_interface>
+      <state_interface name="velocity"/>
+    </joint>
+    <joint name="robotiq_85_right_knuckle_joint">
+      <param name="mimic">robotiq_85_left_knuckle_joint</param>
+      <param name="multiplier">1.0</param>
+      <command_interface name="position"/>
+      <state_interface name="position"/>
+      <state_interface name="velocity"/>
+    </joint>
+    <joint name="robotiq_85_left_inner_knuckle_joint">
+      <param name="mimic">robotiq_85_left_knuckle_joint</param>
+      <param name="multiplier">1.0</param>
+      <command_interface name="position"/>
+      <state_interface name="position"/>
+      <state_interface name="velocity"/>
+    </joint>
+    <joint name="robotiq_85_right_inner_knuckle_joint">
+      <param name="mimic">robotiq_85_left_knuckle_joint</param>
+      <param name="multiplier">1.0</param>
+      <command_interface name="position"/>
+      <state_interface name="position"/>
+      <state_interface name="velocity"/>
+    </joint>
+    <joint name="robotiq_85_left_finger_tip_joint">
+      <param name="mimic">robotiq_85_left_knuckle_joint</param>
+      <param name="multiplier">-1.0</param>
+      <command_interface name="position"/>
+      <state_interface name="position"/>
+      <state_interface name="velocity"/>
+    </joint>
+    <joint name="robotiq_85_right_finger_tip_joint">
+      <param name="mimic">robotiq_85_left_knuckle_joint</param>
+      <param name="multiplier">-1.0</param>
+      <command_interface name="position"/>
+      <state_interface name="position"/>
       <state_interface name="velocity"/>
     </joint>
