Commit message: feat: Add a ZED2 camera to environment and RViz

File: ros2_ws/src/use_case_sim/urdf/assembly_env.urdf.xacro (robot description, xacro)
@@ -54,4 +54,46 @@
   <gazebo reference="prism2_link"><material>Gazebo/White</material></gazebo>
   <gazebo reference="rear_plate_link"><material>Gazebo/DarkGrey</material></gazebo>
+  <joint name="world_to_camera" type="fixed">
+    <parent link="world"/>
+    <child link="camera_link"/>
+    <origin xyz="2.0 0 2.5" rpy="0 0.9 3.14159"/>
+  </joint>
+  <link name="camera_link">
+    <visual><geometry><box size="0.03 0.12 0.03"/></geometry><material name="black"><color rgba="0.1 0.1 0.1 1"/></material></visual>
+    <collision><geometry><box size="0.03 0.12 0.03"/></geometry></collision>
+    <inertial><mass value="0.2"/><inertia ixx="0.0001" ixy="0" ixz="0" iyy="0.0001" iyz="0" izz="0.0001"/></inertial>
+  </link>
+  <joint name="camera_optical_joint" type="fixed">
+    <parent link="camera_link"/>
+    <child link="camera_optical_frame"/>
+    <origin xyz="0 0 0" rpy="-1.5708 0 -1.5708"/>
+  </joint>
+  <link name="camera_optical_frame"/>
+  <gazebo reference="camera_link">
+    <material>Gazebo/FlatBlack</material>
+    <sensor type="depth" name="zed2_camera_sensor">
+      <update_rate>30.0</update_rate>
+      <camera>
+        <horizontal_fov>1.5</horizontal_fov>
+        <image>
+          <width>1280</width>
+          <height>720</height>
+          <format>R8G8B8</format>
+        </image>
+        <clip>
+          <near>0.1</near>
+          <far>10.0</far>
+        </clip>
+      </camera>
+      <plugin name="camera_plugin" filename="libgazebo_ros_camera.so">
+        <ros>
+          <namespace>zed2</namespace>
+        </ros>
+        <frame_name>camera_optical_frame</frame_name>
+        <min_depth>0.2</min_depth>
+        <max_depth>10.0</max_depth>
+      </plugin>
+    </sensor>
+  </gazebo>
   <xacro:include filename="$(find robotiq_description)/urdf/robotiq_2f_85_macro.urdf.xacro"/>
   <xacro:robotiq_gripper name="RobotiqGripper" prefix="" parent="tool0" include_ros2_control="false">
